Commit message: change package name

File: urdf/braccio_arm.urdf (robot description, URDF)
Before this commit: robot visual, 8 links, 7 joints
Links:
- link braccio_base_link: geometry visual mesh filename=package://ros_braccio_opencv_detect_picknplace/stl/braccio_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 scale=0.001 0.001 0.001
- link elbow_link: geometry visual mesh filename=package://ros_braccio_opencv_detect_picknplace/stl/braccio_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 scale=0.001 0.001 0.001
- link left_gripper_link: geometry visual mesh filename=package://ros_braccio_opencv_detect_picknplace/stl/braccio_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 scale=0.001 0.001 0.001
- link right_gripper_link: geometry visual mesh filename=package://ros_braccio_opencv_detect_picknplace/stl/braccio_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 scale=0.001 0.001 0.001
- link shoulder_link: geometry visual mesh filename=package://ros_braccio_opencv_detect_picknplace/stl/braccio_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 scale=0.001 0.001 0.001
- link wrist_pitch_link: geometry visual mesh filename=package://ros_braccio_opencv_detect_picknplace/stl/braccio_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 scale=0.001 0.001 0.001
- link wrist_roll_link: geometry visual mesh filename=package://ros_braccio_opencv_detect_picknplace/stl/braccio_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 scale=0.001 0.001 0.001

Commit message: better name

File: urdf/braccio_arm.urdf (robot description, URDF)
Before this commit: robot visual, 8 links, 7 joints
Links:
- link braccio_base_link: geometry visual mesh filename=package://ros_braccio_opencv_obj_detect_grab/stl/braccio_ba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 scale=0.001 0.001 0.001
- link elbow_link: geometry visual mesh filename=package://ros_braccio_opencv_obj_detect_grab/stl/braccio_el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 scale=0.001 0.001 0.001
- link left_gripper_link: geometry visual mesh filename=package://ros_braccio_opencv_obj_detect_grab/stl/braccio_le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 scale=0.001 0.001 0.001
- link right_gripper_link: geometry visual mesh filename=package://ros_braccio_opencv_obj_detect_grab/stl/braccio_ri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 scale=0.001 0.001 0.001
- link shoulder_link: geometry visual mesh filename=package://ros_braccio_opencv_obj_detect_grab/stl/braccio_sh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 scale=0.001 0.001 0.001
- link wrist_pitch_link: geometry visual mesh filename=package://ros_braccio_opencv_obj_detect_grab/stl/braccio_wr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 scale=0.001 0.001 0.001
- link wrist_roll_link: geometry visual mesh filename=package://ros_braccio_opencv_obj_detect_grab/stl/braccio_wr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 scale=0.001 0.001 0.001

Commit message: switch to su_chef

File: urdf/braccio_arm.urdf (robot description, URDF)
Before this commit: robot visual, 8 links, 7 joints
Links:
- link base_link: mass None -> 1; geometry collision cylinder length=0.01 radius=.053; visual cylinder length=0.01 radius=.053
- link braccio_base_link: mass None -> 0.01; geometry collision mesh filename=package://su_chef/stl/braccio_base.stl scale=0.001 0.001 0.001; visual mesh filename=package://su_chef/stl/braccio_base.stl scale=0.001 0.001 0.001
- link elbow_link: mass None -> 0.01; geometry collision mesh filename=package://su_chef/stl/braccio_elbow.stl scale=0.001 0.001 0.001; visual mesh filename=package://su_chef/stl/braccio_elbow.stl scale=0.001 0.001 0.001
- link left_gripper_link: mass None -> 0.01; geometry collision mesh filename=package://su_chef/stl/braccio_left_gripper.stl scale=0.001 0.001 0.001; visual mesh filename=package://su_chef/stl/braccio_left_gripper.stl scale=0.001 0.001 0.001
- link right_gripper_link: mass None -> 0.01; geometry collision mesh filename=package://su_chef/stl/braccio_right_gripper.stl scale=0.001 0.001 0.001; visual mesh filename=package://su_chef/stl/braccio_right_gripper.stl scale=0.001 0.001 0.001
- link shoulder_link: mass None -> 0.01; geometry collision mesh filename=package://su_chef/stl/braccio_shoulder.stl scale=0.001 0.001 0.001; visual mesh filename=package://su_chef/stl/braccio_shoulder.stl scale=0.001 0.001 0.001
- link wrist_pitch_link: mass None -> 0.01; geometry collision mesh filename=package://su_chef/stl/braccio_wrist_pitch.stl scale=0.001 0.001 0.001; visual mesh filename=package://su_chef/stl/braccio_wrist_pitch.stl scale=0.001 0.001 0.001
- link wrist_roll_link: mass None -> 0.01; geometry collision mesh filename=package://su_chef/stl/braccio_wrist_roll.stl scale=0.001 0.001 0.001; visual mesh filename=package://su_chef/stl/braccio_wrist_roll.stl scale=0.001 0.001 0.001
